File: pcb/MOD65.kicad_sch (KiCad schematic)
At the start: 33 parts, among them J1 UD, J2 OLED, J3 LEDs, J4 Switch, SW68 RESET, SW69 BOOT, U1 Flash, U2 V Reg, U3 RP2040, Y1 Crystal

Commit message: oki
Parts:
- renumbered SW68 to BTN1, SW69 to BTN2
Other:
- company: pioz -> umbacos
- title: aryess -> MOD65
Changed lines of the file:
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@@
 	(paper "A4")
 	(title_block
-		(title "aryess")
+		(title "MOD65")
 		(date "2025-01-20")
 		(rev "2")
-		(company "pioz")
+		(company "umbacos")
 	)
 	(text "Decoupling 1V1 lines"
@@
 		(on_board yes)
 		(dnp no)
-		(property "Reference" "SW68"
+		(property "Reference" "BTN1"
 			(at 204.47 102.87 0)
 			(effects
@@
 			(project ""
 				(path "/b0797d7c-f6aa-44ba-bae5-ddfe355aa8cb"
-					(reference "SW68")
+					(reference "BTN1")
 					(unit 1)
 				)
@@
 		(on_board yes)
 		(dnp no)
-		(property "Reference" "SW69"
+		(property "Reference" "BTN2"
 			(at 245.11 102.87 0)
 			(effects
@@
 			(project "cutlass"
 				(path "/b0797d7c-f6aa-44ba-bae5-ddfe355aa8cb"
-					(reference "SW69")
+					(reference "BTN2")
 					(unit 1)
 				)
