File: pcb/leds.kicad_sch (KiCad schematic)
At the start: 67 parts

Commit message: oki
Other:
- company: pioz -> umbacos
- title: cutlass -> MOD65
Changed lines of the file:
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@@
 	(paper "A4")
 	(title_block
-		(title "cutlass")
+		(title "MOD65")
 		(date "2025-02-04")
 		(rev "1")
-		(company "pioz")
+		(company "umbacos")
 	)
 	(junction

Commit message: JLCPCB 1
Parts:
- added LED68: SK6812MINI-E, PCM_marbastlib-various:LED_6028R, symbol PCM_marbastlib-various:SK6812MINI-E
Connections:
- net +5V: now also LED68.1 (VDD)
- net GND: now also LED68.4 (VSS)
- net at LED63.3 (DIN): now also LED68.2 (DOUT); no longer LED62.2 (DOUT)
- new net: LED62.2 (DOUT), LED68.3 (DIN)
Changed lines of the file:
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@@
+	)
+	(junction
+		(at 162.56 129.54)
+		(diameter 0)
+		(color 0 0 0 0)
 	)
 	(junction
@@
 	(wire
 		(pts
+			(xy 162.56 129.54) (xy 177.8 129.54)
+		)
+		(stroke
+			(width 0)
+			(type default)
+		)
+	)
+	(wire
+		(pts
 			(xy 254 68.58) (xy 276.86 68.58)
 		)
@@
 	(wire
 		(pts
-			(xy 124.46 121.92) (xy 170.18 121.92)
-		)
-		(stroke
-			(width 0)
-			(type default)
-		)
-	)
-	(wire
-		(pts
 			(xy 238.76 68.58) (xy 254 68.58)
 		)
@@
 	(wire
 		(pts
+			(xy 124.46 121.92) (xy 154.94 121.92)
+		)
+		(stroke
+			(width 0)
+			(type default)
+		)
+	)
+	(wire
+		(pts
 			(xy 116.84 68.58) (xy 132.08 68.58)
 		)
@@
 	(wire
 		(pts
-			(xy 116.84 129.54) (xy 177.8 129.54)
+			(xy 116.84 129.54) (xy 162.56 129.54)
 		)
 		(stroke
@@
 					(unit 1)
 				)
+			)
+		)
+	)
+	(symbol
+		(lib_id "PCM_marbastlib-various:SK6812MINI-E")
+		(at 162.56 121.92 0)
+		(unit 1)
+		(exclude_from_sim no)
+		(in_bom yes)
+		(on_board yes)
+		(dnp no)
+		(fields_autoplaced yes)
+		(property "Reference" "LED68"
+			(at 176.53 115.6014 0)
+			(effects
+				(font
+					(size 1.27 1.27)
+				)
+			)
+		)
+		(property "Value" "SK6812MINI-E"
+			(at 176.53 118.1414 0)
+			(effects
+				(font
+					(size 1.27 1.27)
+				)
+			)
+		)
+		(property "Footprint" "PCM_marbastlib-various:LED_6028R"
+			(at 162.56 121.92 0)
+			(effects
+				(font
+					(size 1.27 1.27)
+				)
+				(hide yes)
+			)
+		)
+		(property "Datasheet" ""
+			(at 162.56 121.92 0)
+			(effects
+				(font
+					(size 1.27 1.27)
+				)
+				(hide yes)
+			)
+		)
+		(property "Description" "Reverse mount adressable LED (WS2812 protocol)"
+			(at 162.56 121.92 0)
+			(effects
+				(font
+					(size 1.27 1.27)
+				)
+				(hide yes)
+			)
+		)
+		(property "Part Number" "SK6812MINI-E"
+			(at 162.56 121.92 0)
+			(effects
+				(font
+					(size 1.27 1.27)
+				)
+				(hide yes)
+			)
+		)
+		(property "JLCPCB Part" "C5149201"
+			(at 162.56 121.92 0)
+			(effects
+				(font
+					(size 1.27 1.27)
+				)
+				(hide yes)
+			)
+		)
+		(property "FT Rotation Offset" ""
+			(at 162.56 121.92 0)
+			(effects
+				(font
+					(size 1.27 1.27)
+				)
+				(hide yes)
+			)
+		)
+		(property "FT Position Offset" ""
+			(at 162.56 121.92 0)
+			(effects
+				(font
+					(size 1.27 1.27)
+				)
+				(hide yes)
+			)
+		)
+		(pin "4"
+		)
+		(pin "1"
+		)
+		(pin "2"
+		)
+		(pin "3"
+		)
+		(instances
+			(project "MOD65"
+				(path "/b0797d7c-f6aa-44ba-bae5-ddfe355aa8cb/58bc1edb-79b5-4355-bdb1-623e0d7b414b"
+					(reference "LED68")
+					(unit 1)
+				)
